File: hardware/ematel_PCB/_autosave-ematel_PCB 3.kicad_sch (KiCad schematic)
At the start: 192 parts, among them J1 BAT, J10 HDR-4x1, J11 IN, J12 Conn_01x02, J13 USB_B_Micro, J14 HDR-2x1, J15 HDR-2x1, J16 HDR-2x1, J17 HDR-2x1, J18 HDR-2x1, J19 HDR-2x1, J2 V_USB, J20 IN, J21 Micro_SD_Card, J22 Conn_01x08, J23 Conn_01x08, J24 HDR-3x1, J25 HDR-3x1, J26 HDR-4x1, J27 HDR-4x1, J28 HDR-4x1, J29 HDR-4x1, J3 HDR-2x1, J30 Conn_01x02, J31 Conn_01x02, J32 Conn_01x02, J4 HDR-2x1, J5 HDR-4x1, J6 HDR-2x1, J7 HDR-2x1, J8 HDR-2x1, J9 HDR-2x1, Q1 Q_PMOS_GSD, Q2 Q_PMOS_GSD, Q3 Q_Dual_NPN_NPN_BRT_E1B1C2E2B2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, SW1 SW_DIP_x02, SW3 SW_DIP_x02, SW4 SW_DIP_x02, U1 TP4056, U10 TPS562200, U11 CH340C, U12 AP2112K-3.3, U13 AP2112K-3.3, U14 AP2112K-3.3, U15 PC817, U16 PC817, U17 PC817, U18 PC817, U19 MCP23008-xSO, U2 MAX3485, U3 DW01, U4 FS8205A, U5 ESP32-WROOM-32D, U6 INA219AxD, U7 INA219AxD, U8 MT3608, U9 RV-8803

Commit message: Actualizacion PCB
Parts:
- removed C13, C15: 0.1u, Capacitor_SMD:C_0805_2012Metric, symbol IoWLabs:C
- removed C14: 10u, Capacitor_SMD:C_0805_2012Metric, symbol IoWLabs:C
- removed C25, C26, C27: 0.1uF, Capacitor_SMD:C_0603_1608Metric, symbol IoWLabs:C
- removed D8: LED, LED_SMD:LED_0603_1608Metric, symbol Device:LED
- removed J10: HDR-4x1, TerminalBlock_Phoenix:TerminalBlock_Phoenix_PT-1,5-4-3.5-H_1x04_P3.50mm_Horizontal, symbol IoWLabsConnectors:HDR-4x1
- removed J16, J17, J7: HDR-2x1, TerminalBlock_Phoenix:TerminalBlock_Phoenix_PT-1,5-2-3.5-H_1x02_P3.50mm_Horizontal, symbol IoWLabsConnectors:HDR-2x1
- removed J19, J9: HDR-2x1, Connector_PinHeader_2.54mm:PinHeader_1x02_P2.54mm_Vertical, symbol IoWLabsConnectors:HDR-2x1
- removed J22: Conn_01x08, Connector_JST:JST_XH_B8B-XH-AM_1x08_P2.50mm_Vertical, symbol Connector_Generic:Conn_01x08
- removed J23: Conn_01x08, Connector_JST:JST_XH_B6B-XH-AM_1x06_P2.50mm_Vertical, symbol Connector_Generic:Conn_01x06
- removed J26, J27, J28, J29: HDR-4x1, TerminalBlock_Phoenix:TerminalBlock_Phoenix_PT-1,5-4-3.5-H_1x04_P3.50mm_Horizontal, symbol IoWLabsConnectors:HDR-3x1
- removed J30, J31, J32: Conn_01x02, Connector_JST:JST_XH_B2B-XH-AM_1x02_P2.50mm_Vertical, symbol Connector_Generic:Conn_01x02
- removed JP10, JP11, JP6, JP8, JP9: SolderJumper_2_Open, Jumper:SolderJumper-2_P1.3mm_Open_RoundedPad1.0x1.5mm, symbol Jumper:SolderJumper_2_Open
- removed R36: 54.9k, Resistor_SMD:R_0603_1608Metric, symbol IoWLabs:RES
- removed R37: 470, Resistor_SMD:R_0603_1608Metric, symbol IoWLabs:RES
- removed R38, R44, R52, R53, R54, R55, R66, R68: 10k, Resistor_SMD:R_0603_1608Metric, symbol IoWLabs:RES
- removed R46, R48, R51, R67, R69, R74, R75, R76: 3.3k, Resistor_SMD:R_0603_1608Metric, symbol IoWLabs:RES
- removed R57, R58, R59, R60, R61, R62, R63, R70, R71, R72, R73: 1k, Resistor_SMD:R_0603_1608Metric, symbol IoWLabs:RES
- removed U10: TPS562200, Package_TO_SOT_SMD:SOT-23-6, symbol Regulator_Switching:TPS562200
- removed U15, U16, U17, U18: PC817, Package_DIP:DIP-4_W7.62mm, symbol Isolator:PC817
- removed U19: MCP23008-xSO, Package_SO:SOIC-18W_7.5x11.6mm_P1.27mm, symbol Interface_Expansion:MCP23008-xSO
- added C14: 220uF, Capacitor_SMD:CP_Elec_8x10.5, symbol Device:C_Polarized
- added C16: 10u, Capacitor_SMD:C_0603_1608Metric, symbol IoWLabs:C
- added C9: 680uF, Capacitor_SMD:CP_Elec_8x10.5, symbol Device:C_Polarized
- added D10: SS34, Diode_SMD:D_SMA, symbol Device:D_Schottky
- added D11: LED, LED_SMD:LED_0603_1608Metric, symbol Device:LED
- added R32: 1k, Resistor_SMD:R_0603_1608Metric, symbol IoWLabs:RES
- added U15: MCP23017_SO, Package_SO:SOIC-28W_7.5x17.9mm_P1.27mm, symbol Interface_Expansion:MCP23017_SO
- added U9: LM2596S-5, Package_TO_SOT_SMD:TO-263-5_TabPin3, symbol Regulator_Switching:LM2596S-5
- C10: renamed from C20; footprint Capacitor_SMD:C_0805_2012Metric -> Capacitor_SMD:C_0603_1608Metric
- C11: renamed from C21; footprint Capacitor_SMD:C_0805_2012Metric -> Capacitor_SMD:C_0603_1608Metric
- C12: renamed from C22; footprint Capacitor_SMD:C_0805_2012Metric -> Capacitor_SMD:C_0603_1608Metric
- C13: renamed from C23; footprint Capacitor_SMD:C_0805_2012Metric -> Capacitor_SMD:C_0603_1608Metric
- C15: renamed from C24; footprint Capacitor_SMD:C_0805_2012Metric -> Capacitor_SMD:C_0603_1608Metric
- C8: renamed from C19; footprint Capacitor_SMD:C_0805_2012Metric -> Capacitor_SMD:C_0603_1608Metric
- J11: renamed from J5; footprint TerminalBlock_Phoenix:TerminalBlock_Phoenix_PT-1,5-4-3.5-H_1x04_P3.50mm_Horizontal -> IoWLabsConnectors:TB-4x1-5P-TH-V
- J12: renamed from J3; footprint TerminalBlock_Phoenix:TerminalBlock_Phoenix_PT-1,5-2-3.5-H_1x02_P3.50mm_Horizontal -> IoWLabsConnectors:Tb-2x1-5p-TH-V
- J14: renamed from J15; footprint TerminalBlock_Phoenix:TerminalBlock_Phoenix_PT-1,5-2-3.5-H_1x02_P3.50mm_Horizontal -> IoWLabsConnectors:Tb-2x1-5p-TH-V
- J16: renamed from J14; footprint TerminalBlock_Phoenix:TerminalBlock_Phoenix_PT-1,5-2-3.5-H_1x02_P3.50mm_Horizontal -> IoWLabsConnectors:Tb-2x1-5p-TH-V
- J2: renamed from J1; footprint TerminalBlock_Phoenix:TerminalBlock_Phoenix_PT-1,5-2-3.5-H_1x02_P3.50mm_Horizontal -> IoWLabsConnectors:Tb-2x1-5p-TH-V
- J4: renamed from J20; footprint TerminalBlock_Phoenix:TerminalBlock_Phoenix_PT-1,5-2-3.5-H_1x02_P3.50mm_Horizontal -> IoWLabsConnectors:Tb-2x1-5p-TH-V
- L2: value 4.7u -> 33uH; footprint Inductor_SMD:L_Bourns_SRP7028A_7.3x6.6mm -> Inductor_SMD:L_12x12mm_H8mm; type (none) -> L40
- R10: renamed from R22; value 10k -> 10K
- R12: renamed from R21; value 10k -> 10K
- R13: renamed from R14; value 10k -> 4.7k
- R14: renamed from R16; value 10k -> 4.7k
- R15: renamed from R23; value 10k -> 10K
- R17: value 10k -> 10K
- R19: renamed from R2; value 1k2 -> 1K2
- R20: renamed from R12; value 1k -> 1K
- R21: renamed from R24; value 7k5 -> 7K5
- R22: renamed from R29; value 1k -> 1K
- R23: renamed from R3; value 12k -> 12K
- R25: renamed from R4; value 30k -> 30K
- R29: renamed from R39; value 10k -> 10K
- R30: renamed from R40; value 12k -> 12K
- R31: renamed from R41; value 30k -> 30K
- R33: renamed from R49; value 10k -> 10K
- R34: renamed from R50; value 10k -> 10K
- R38: renamed from R26; value 10k -> 10K
- R39: renamed from R27; value 10k -> 10K
- R43: renamed from R33; value 10k -> 2.2k
- R44: renamed from R34; value 10k -> 2.2k
- R7: renamed from R20; value 10k -> 10K
- R8: renamed from R13; value 10k -> 4.7k
- R9: renamed from R15; value 10k -> 4.7k
- renumbered C6 to C1, C3 to C17, C4 to C18, C10 to C19, C7 to C2, C11 to C20, C12 to C21, C17 to C22, C18 to C23, C16 to C24, C8 to C3, C5 to C4, C2 to C5, C1 to C6, C9 to C7, D3 to D12, D7 to D13, D6 to D3, D10 to D6, D11 to D7, D12 to D8, H3 to H2, H2 to H3, J2 to J1, J21 to J10, J4 to J13, J18 to J15, J13 to J17, J6 to J3, J25 to J5, J24 to J6, J11 to J7, J12 to J9, JP7 to JP6, R9 to R1, R19 to R11, R1 to R16, R10 to R18, R5 to R2, R25 to R24, R56 to R26, R64 to R27, R65 to R28, R6 to R3, R11 to R35, R30 to R36, R28 to R37, R7 to R4, R35 to R40, R31 to R41, R32 to R42, R42 to R46, R43 to R47, R47 to R48, R8 to R5, R18 to R6, U2 to U1, U13 to U10, U14 to U11, U5 to U12, U9 to U13, U11 to U14, U6 to U2, U7 to U3, U3 to U4, U1 to U5, U8 to U6, U4 to U7, U12 to U8
Connections:
- net 12V_IN: now also R30.2
- net 420_VDD_ch2: now also J14.1; no longer J16.1
- net 420_VSS_ch2: no longer J16.2
- net GND: now also C14.2, C16.2, C9.2, D10.2 (A), D11.1 (K), U9.3 (GND), U9.5 (~{ON}/OFF)
- net RS485_A_ch2: no longer R1.2, U1.6 (A)
- net RS485_B_ch2: no longer R1.1, U1.7 (B)
- net SCL: now also U15.12 (SCK); no longer R43.2
- net SDA: now also U15.13 (SDA); no longer R44.2
- net SD_CS: no longer U12.29 (IO5)
- net SENSOR 2: now also U12.29 (IO5)
- net VIN_12V: now also C9.1, U9.1 (VIN); no longer R30.2
- net VIN_5V: now also C14.1, C16.1, R32.2, U9.4 (FB)
- net at L2.1: now also D10.1 (K), U9.2 (OUT)
- net 420_sens_ch1+ renamed 420_VDD_ch1+
- net 420_sens_ch2+ renamed 420_VDD_ch2+
- net 420_VDD_ch2+: no longer J14.1
- net IO2 renamed IO2 GPB
- net VRFID_3V3 renamed VGPS_3V3
- new net: D11.2 (A), R32.1
- new net 420_sens_ch2_: J16.1
- new net 420_sens_ch2_+: J16.2
- new net Data_A: R1.2, U1.6 (A)
- new net Data_B: R1.1, U1.7 (B)
- new net scl: R43.2
- new net sda: R44.2
Other:
- note added: "CONECTORES"
- note added: "GPS supply - LED"
- note added: "Lista de pines: ---------------- io0 - BOOT io1 - Tx io2 - LED status io3 - Rx io4 - DO_LORA io5 - SD_CS io12 - SPI2_MISO io13 - SPI2_MOSI io14 - SPI2_CLK io15 - LORA_CS io16 - D1_LORA io17 - RST_LORA io18 - SPI1_CLK io19 - SPI1_MISO io21 - SDA/CS io22 - SCL/SCK io23 - SPI1_MOSI io25 - RST_GPS i026 - RGB_PIN io27 - EN_VDL io32 - EN_VS io33 - io34 - BTN1 io35 - BTN2 io36 - V_AUTO_LVL io39 - BAT_LVL"
- note added: "Power CH2"
- note added: "Sensor CH2"
- note removed: "B1"
- note removed: "B2"
- note removed: "B3"
- note removed: "CONECTORES GPIO EXT"
- note removed: "CONECTORES PROTOCOLOS"
- note removed: "CONECTORES SENSORES Y OPTOCUPLAS"
- note removed: "DEBOUNCERS"
- note removed: "Lista de pines: ---------------- io0 - BOOT io1 - Tx io2 - LED status io3 - Rx io4 - SENSOR 1 io5 - SD/CS io12 - KR2 io13 - KR1 io14 - KR3 io15 - RS485_EN io16 - 485_TX io17 - 485_RX io18 - SPI1_CLK io19 - SPI1_MISO io21 - SDA io22 - SCL io23 - SPI1_MOSI io25 - KC2 i026 - KC1 io27 - KR4 io32 - KC4 io33 - KC3 io34 - SENSOR 3 io35 - SENSOR 4 io36 - V_AUTO_LVL io39 - BAT_LVL"
- note removed: "MCP23008 IO EXTENSOR"
- note removed: "Power CH2/CH1"
- note removed: "RFID"
- note removed: "RFID AGREGAR COMO CONECTOR-> listo AGREGAR CH1 420 Y 485 -> listo IMPLEMENTAR OPTOCUPLA -> listo SE CAMBIA MCP32017 POR MCP23008"
- note removed: "RFID supply - LED"
- note removed: "Sensor CH2/CH1"
- note removed: "V_out = 0.765(R20/R21 + 1)"
- moved on the sheet: BT1, C1, C19, C2, C20, C21, C22, C23, C24, D13, D9, F1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
