File: hardware/ematel_PCB/_autosave-ematel_PCB 8.kicad_sch (KiCad schematic)
At the start: 192 parts, among them J1 BAT, J10 HDR-4x1, J11 IN, J12 Conn_01x02, J13 USB_B_Micro, J14 HDR-2x1, J15 HDR-2x1, J16 HDR-2x1, J17 HDR-2x1, J18 HDR-2x1, J19 HDR-2x1, J2 V_USB, J20 IN, J21 Micro_SD_Card, J22 Conn_01x08, J23 Conn_01x08, J24 HDR-3x1, J25 HDR-3x1, J26 HDR-4x1, J27 HDR-4x1, J28 HDR-4x1, J29 HDR-4x1, J3 HDR-2x1, J30 Conn_01x02, J31 Conn_01x02, J32 Conn_01x02, J4 HDR-2x1, J5 HDR-4x1, J6 HDR-2x1, J7 HDR-2x1, J8 HDR-2x1, J9 HDR-2x1, Q1 Q_PMOS_GSD, Q2 Q_PMOS_GSD, Q3 Q_Dual_NPN_NPN_BRT_E1B1C2E2B2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, SW1 SW_DIP_x02, SW3 SW_DIP_x02, SW4 SW_DIP_x02, U1 TP4056, U10 TPS562200, U11 CH340C, U12 AP2112K-3.3, U13 AP2112K-3.3, U14 AP2112K-3.3, U15 PC817, U16 PC817, U17 PC817, U18 PC817, U19 MCP23008-xSO, U2 MAX3485, U3 DW01, U4 FS8205A, U5 ESP32-WROOM-32D, U6 INA219AxD, U7 INA219AxD, U8 MT3608, U9 RV-8803

Commit message: Actualizacion PCB
Parts:
- removed C13: 0.1u, Capacitor_SMD:C_0805_2012Metric, symbol IoWLabs:C
- removed C14: 10u, Capacitor_SMD:C_0805_2012Metric, symbol IoWLabs:C
- removed D8: LED, LED_SMD:LED_0603_1608Metric, symbol Device:LED
- removed J10: HDR-4x1, TerminalBlock_Phoenix:TerminalBlock_Phoenix_PT-1,5-4-3.5-H_1x04_P3.50mm_Horizontal, symbol IoWLabsConnectors:HDR-4x1
- removed J16, J17, J7: HDR-2x1, TerminalBlock_Phoenix:TerminalBlock_Phoenix_PT-1,5-2-3.5-H_1x02_P3.50mm_Horizontal, symbol IoWLabsConnectors:HDR-2x1
- removed J19, J9: HDR-2x1, Connector_PinHeader_2.54mm:PinHeader_1x02_P2.54mm_Vertical, symbol IoWLabsConnectors:HDR-2x1
- removed J22: Conn_01x08, Connector_JST:JST_XH_B8B-XH-AM_1x08_P2.50mm_Vertical, symbol Connector_Generic:Conn_01x08
- removed J23: Conn_01x08, Connector_JST:JST_XH_B6B-XH-AM_1x06_P2.50mm_Vertical, symbol Connector_Generic:Conn_01x06
- removed JP6, JP8: SolderJumper_2_Open, Jumper:SolderJumper-2_P1.3mm_Open_RoundedPad1.0x1.5mm, symbol Jumper:SolderJumper_2_Open
- removed R36: 54.9k, Resistor_SMD:R_0603_1608Metric, symbol IoWLabs:RES
- removed R37: 470, Resistor_SMD:R_0603_1608Metric, symbol IoWLabs:RES
- removed R44: 10k, Resistor_SMD:R_0603_1608Metric, symbol IoWLabs:RES
- removed R46, R48, R51: 3.3k, Resistor_SMD:R_0603_1608Metric, symbol IoWLabs:RES
- removed R60, R61, R62, R63, R70, R71, R72, R73: 1k, Resistor_SMD:R_0603_1608Metric, symbol IoWLabs:RES
- removed U10: TPS562200, Package_TO_SOT_SMD:SOT-23-6, symbol Regulator_Switching:TPS562200
- removed U15, U16, U17, U18: PC817, Package_DIP:DIP-4_W7.62mm, symbol Isolator:PC817
- removed U19: MCP23008-xSO, Package_SO:SOIC-18W_7.5x11.6mm_P1.27mm, symbol Interface_Expansion:MCP23008-xSO
- added C13: 680uF, Capacitor_SMD:CP_Elec_8x10.5, symbol Device:C_Polarized
- added C14: 220uF, Capacitor_SMD:CP_Elec_8x10.5, symbol Device:C_Polarized
- added D8: SS34, Diode_SMD:D_SMA, symbol Device:D_Schottky
- added D9: LED, LED_SMD:LED_0603_1608Metric, symbol Device:LED
- added J15: Conn_01x04, Connector_JST:JST_XH_B3B-XH-A_1x03_P2.50mm_Vertical, symbol Connector_Generic:Conn_01x04
- added J16: Conn_01x08, Connector_JST:JST_XH_B3B-XH-A_1x03_P2.50mm_Vertical, symbol Connector_Generic:Conn_01x08
- added R53, R54, R55: 10k2, Resistor_SMD:R_0603_1608Metric, symbol IoWLabs:RES
- added R56, R57, R58, R59: 3k3, Resistor_SMD:R_0603_1608Metric, symbol IoWLabs:RES
- added R67: 3.3k, Resistor_SMD:R_0603_1608Metric, symbol IoWLabs:RES
- added U10: LM2596S-5, Package_TO_SOT_SMD:TO-263-5_TabPin3, symbol Regulator_Switching:LM2596S-5
- added U15: MCP23017_SO, Package_SO:SOIC-28W_7.5x17.9mm_P1.27mm, symbol Interface_Expansion:MCP23017_SO
- C15: value 0.1u -> 10u; footprint Capacitor_SMD:C_0805_2012Metric -> Capacitor_SMD:C_0603_1608Metric
- J1, J3: footprint TerminalBlock_Phoenix:TerminalBlock_Phoenix_PT-1,5-2-3.5-H_1x02_P3.50mm_Horizontal -> IoWLabsConnectors:Tb-2x1-5p-TH-V
- J14: renamed from J20; footprint TerminalBlock_Phoenix:TerminalBlock_Phoenix_PT-1,5-2-3.5-H_1x02_P3.50mm_Horizontal -> IoWLabsConnectors:Tb-2x1-5p-TH-V
- J20: renamed from J26; footprint TerminalBlock_Phoenix:TerminalBlock_Phoenix_PT-1,5-4-3.5-H_1x04_P3.50mm_Horizontal -> IoWLabsConnectors:TB-4x1-5P-TH-V
- J21: renamed from J27; footprint TerminalBlock_Phoenix:TerminalBlock_Phoenix_PT-1,5-4-3.5-H_1x04_P3.50mm_Horizontal -> IoWLabsConnectors:TB-4x1-5P-TH-V
- J22: renamed from J28; footprint TerminalBlock_Phoenix:TerminalBlock_Phoenix_PT-1,5-4-3.5-H_1x04_P3.50mm_Horizontal -> IoWLabsConnectors:TB-4x1-5P-TH-V
- J23: renamed from J29; footprint TerminalBlock_Phoenix:TerminalBlock_Phoenix_PT-1,5-4-3.5-H_1x04_P3.50mm_Horizontal -> IoWLabsConnectors:TB-4x1-5P-TH-V
- J24: renamed from J30; footprint Connector_JST:JST_XH_B2B-XH-AM_1x02_P2.50mm_Vertical -> Connector_JST:JST_XH_B3B-XH-A_1x03_P2.50mm_Vertical
- J25: renamed from J31; footprint Connector_JST:JST_XH_B2B-XH-AM_1x02_P2.50mm_Vertical -> Connector_JST:JST_XH_B3B-XH-A_1x03_P2.50mm_Vertical
- J26: renamed from J32; footprint Connector_JST:JST_XH_B2B-XH-AM_1x02_P2.50mm_Vertical -> Connector_JST:JST_XH_B3B-XH-A_1x03_P2.50mm_Vertical
- J5: footprint TerminalBlock_Phoenix:TerminalBlock_Phoenix_PT-1,5-4-3.5-H_1x04_P3.50mm_Horizontal -> IoWLabsConnectors:TB-4x1-5P-TH-V
- J7: renamed from J14; footprint TerminalBlock_Phoenix:TerminalBlock_Phoenix_PT-1,5-2-3.5-H_1x02_P3.50mm_Horizontal -> IoWLabsConnectors:Tb-2x1-5p-TH-V
- J8: renamed from J15; footprint TerminalBlock_Phoenix:TerminalBlock_Phoenix_PT-1,5-2-3.5-H_1x02_P3.50mm_Horizontal -> IoWLabsConnectors:Tb-2x1-5p-TH-V
- L2: value 4.7u -> 33uH; footprint Inductor_SMD:L_Bourns_SRP7028A_7.3x6.6mm -> Inductor_SMD:L_12x12mm_H8mm; type (none) -> L40
- R38: value 10k -> 1k
- R52: value 10k -> 10k2
- renumbered C11 to C10, C9 to C11, C10 to C9, D9 to D10, D10 to D11, D11 to D12, D12 to D13, J18 to J10, J21 to J17, J24 to J18, J25 to J19, J8 to J9, JP7 to JP6, JP9 to JP7, JP10 to JP8, JP11 to JP9, Q3 to Q2, Q2 to Q3, R26 to R24, R27 to R25, R28 to R26, R24 to R27, R25 to R28, R49 to R36, R50 to R37, R42 to R40, R40 to R41, R41 to R42, R45 to R44, R47 to R45, R53 to R46, R54 to R47, R55 to R48, R57 to R49, R58 to R50, R59 to R51, R56 to R60, R64 to R61, R65 to R62, R66 to R63, R68 to R64, R67 to R65, R69 to R66, R74 to R68, R75 to R69, R76 to R70
Connections:
- net +3V3: now also R67.2, U15.9 (VDD)
- net 420_VDD_ch2: now also J8.1; no longer J7.1
- net 420_VSS_ch2: no longer J7.2
- net A0: now also U15.15 (A0)
- net A1: now also U15.16 (A1)
- net A2: now also U15.17 (A2)
- net GND: now also C13.2, C14.2, D8.2 (A), D9.1 (K), R56.1, R57.1, R58.1, R59.1, U10.3 (GND), U10.5 (~{ON}/OFF), U15.10 (VSS); no longer R38.2
- net GPA0: now also U15.21 (GPA0)
- net GPA1: now also U15.22 (GPA1)
- net GPA2: now also U15.23 (GPA2)
- net GPA4: now also J15.1 (Pin_1), U15.25 (GPA4)
- net GPA5: now also J15.2 (Pin_2), U15.26 (GPA5)
- net GPA6: now also J15.3 (Pin_3), U15.27 (GPA6)
- net GPA7: now also J15.4 (Pin_4), U15.28 (GPA7)
- net INTA: now also U15.20 (INTA)
- net MCP_RESET: now also U15.18 (~{RESET})
- net RS485_A_ch2: no longer R9.2, U2.6 (A)
- net RS485_B_ch2: no longer R9.1, U2.7 (B)
- net S1_IN: now also R52.1
- net S2_IN: now also R53.1
- net S3_IN: now also R54.1
- net S4_IN: now also R55.1
- net SCL: now also R64.1; no longer R63.1
- net SDA: now also R63.1; no longer R52.2, R64.1
- net SENSOR 1: now also R52.2, R56.2
- net SENSOR 2: now also R53.2, R57.2, U15.24 (GPA3)
- net SENSOR 3: now also R54.2, R58.2
- net SENSOR 4: now also R55.2, R59.2
- net VIN_12V: now also C13.1, U10.1 (VIN); no longer C15.1
- net VIN_5V: now also C15.1, R38.2, C14.1, U10.4 (FB); no longer R38.1
- net at L2.1: now also D8.1 (K), U10.2 (OUT)
- net at R64.2: now also U15.12 (SCK)
- net at R63.2: now also U15.13 (SDA)
- net 420_sens_ch1+ renamed 420_VDD_ch1+
- net 420_sens_ch2+ renamed 420_VDD_ch2+
- net 420_VDD_ch2+: no longer J8.1
- net VRFID_3V3 renamed VGPS_3V3
- new net: D9.2 (A), R38.1
- new net 420_sens_ch2_: J7.1
- new net 420_sens_ch2_+: J7.2
- new net Data_A: R9.2, U2.6 (A)
- new net Data_B: R9.1, U2.7 (B)
- new net GPB0: J16.1 (Pin_1), U15.1 (GPB0)
- new net GPB1: J16.2 (Pin_2), U15.2 (GPB1)
- new net GPB2: J16.3 (Pin_3), U15.3 (GPB2)
- new net GPB3: J16.4 (Pin_4), U15.4 (GPB3)
- new net GPB4: J16.5 (Pin_5), U15.5 (GPB4)
- new net GPB5: J16.6 (Pin_6), U15.6 (GPB5)
- new net GPB6: J16.7 (Pin_7), U15.7 (GPB6)
- new net GPB7: J16.8 (Pin_8), U15.8 (GPB7)
- new net INTB: R67.1, U15.19 (INTB)
Other:
- note added: "CONECTORES SENSORES"
- note added: "GPS supply - LED"
- note added: "MCP23017 IO EXTENSOR"
- note added: "Power CH2"
- note added: "Sensor CH2"
- note removed: "CONECTORES SENSORES Y OPTOCUPLAS"
- note removed: "MCP23008 IO EXTENSOR"
- note removed: "Power CH2/CH1"
- note removed: "RFID"
- note removed: "RFID AGREGAR COMO CONECTOR-> listo AGREGAR CH1 420 Y 485 -> listo IMPLEMENTAR OPTOCUPLA -> listo SE CAMBIA MCP32017 POR MCP23008"
- note removed: "RFID supply - LED"
- note removed: "Sensor CH2/CH1"
- note removed: "V_out = 0.765(R20/R21 + 1)"
- moved on the sheet: C10, C16, C25, C26, C27, C9, D10, F1, J10, J11, J13, J14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
