File: hardware/ematel_PCB/ematel_PCB.kicad_pcb (KiCad board)
At the start: 2 copper layers, 175 parts, among them J1 BAT, J10 HDR-2x1, J11 IN, J12 Conn_01x02, J13 USB_B_Micro, J14 IN, J15 Conn_01x04, J16 Conn_01x08, J17 Micro_SD_Card, J18 HDR-3x1, J19 HDR-3x1, J2 V_USB, J20 HDR-4x1, J21 HDR-4x1, J22 HDR-4x1, J23 HDR-4x1, J24 Conn_01x02, J25 Conn_01x02, J26 Conn_01x02, J3 HDR-2x1, J4 HDR-2x1, J5 HDR-4x1, J6 HDR-2x1, J7 HDR-2x1, J8 HDR-2x1, J9 HDR-2x1, Q1 Q_PMOS_GSD, Q2 Q_Dual_NPN_NPN_BRT_E1B1C2E2B2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, Q3 Q_PMOS_GSD, SW1 SW_DIP_x02, SW3 SW_DIP_x02, SW4 SW_DIP_x02, U1 TP4056, U10 LM2596S-5, U11 CH340C, U12 AP2112K-3.3, U13 AP2112K-3.3, U14 AP2112K-3.3, U15 MCP23017_SO, U2 MAX3485, U3 DW01, U4 FS8205A, U5 ESP32-WROOM-32D, U6 INA219AxD, U7 INA219AxD, U8 MT3608, U9 RV-8803

Commit message: Actualizacion PCB
Parts:
- removed D13: LED, LED_SMD:LED_0603_1608Metric
- added J27: HDR-4x1, TerminalBlock_Phoenix:TerminalBlock_Phoenix_PT-1,5-4-3.5-H_1x04_P3.50mm_Horizontal, F.Cu at (154.7, 129.7)
- added J28: HDR-4x1, TerminalBlock_Phoenix:TerminalBlock_Phoenix_PT-1,5-4-3.5-H_1x04_P3.50mm_Horizontal, F.Cu at (169.7, 129.7)
- added J29: HDR-4x1, TerminalBlock_Phoenix:TerminalBlock_Phoenix_PT-1,5-4-3.5-H_1x04_P3.50mm_Horizontal, F.Cu at (184.8, 129.7)
- added J30: Conn_01x02, Connector_JST:JST_XH_B2B-XH-AM_1x02_P2.50mm_Vertical, F.Cu at (106.8, 130.4)
- added J31: Conn_01x02, Connector_JST:JST_XH_B2B-XH-AM_1x02_P2.50mm_Vertical, F.Cu at (115.3, 130.4)
- added J32: Conn_01x02, Connector_JST:JST_XH_B2B-XH-AM_1x02_P2.50mm_Vertical, F.Cu at (123.8, 130.4)
- added JP10: SolderJumper_2_Open, Jumper:SolderJumper-2_P1.3mm_Open_RoundedPad1.0x1.5mm, F.Cu at (77.5, 115.4)
- added JP11: SolderJumper_2_Open, Jumper:SolderJumper-2_P1.3mm_Open_RoundedPad1.0x1.5mm, F.Cu at (77.5, 112.9)
- added R71: 1k, Resistor_SMD:R_0603_1608Metric, F.Cu at (143.3, 118.5)
- added R72: 1k, Resistor_SMD:R_0603_1608Metric, F.Cu at (159.1, 118.6)
- added R73: 1k, Resistor_SMD:R_0603_1608Metric, F.Cu at (174.9, 118.6)
- added R74: 3.3k, Resistor_SMD:R_0603_1608Metric, F.Cu at (165.4, 42.2)
- added R75: 3.3k, Resistor_SMD:R_0603_1608Metric, F.Cu at (165.4, 40.6)
- added R76: 3.3k, Resistor_SMD:R_0603_1608Metric, F.Cu at (165.4, 39.1)
- added U16: PC817, Package_DIP:DIP-4_W7.62mm, F.Cu at (145.2, 118.6)
- added U17: PC817, Package_DIP:DIP-4_W7.62mm, F.Cu at (161.0, 118.6)
- added U18: PC817, Package_DIP:DIP-4_W7.62mm, F.Cu at (176.8, 118.6)
- added U19: MCP23008-xSO, Package_SO:SOIC-18W_7.5x11.6mm_P1.27mm, F.Cu at (173.0, 41.4)
- C11: value 22u -> 100n; footprint Capacitor_SMD:C_0805_2012Metric -> Capacitor_SMD:C_0603_1608Metric
- C13: value 680uF -> 0.1u; footprint Capacitor_SMD:CP_Elec_8x10.5 -> Capacitor_SMD:C_0805_2012Metric
- C14: value 220uF -> 10u; footprint Capacitor_SMD:CP_Elec_8x10.5 -> Capacitor_SMD:C_0805_2012Metric
- C15: value 10u -> 0.1u; footprint Capacitor_SMD:C_0603_1608Metric -> Capacitor_SMD:C_0805_2012Metric
- C9: value 100n -> 22u; footprint Capacitor_SMD:C_0603_1608Metric -> Capacitor_SMD:C_0805_2012Metric
- D10: value D_Schottky -> LED; footprint Diode_SMD:D_SMA -> LED_SMD:LED_0603_1608Metric
- D8: value SS34 -> LED; footprint Diode_SMD:D_SMA -> LED_SMD:LED_0603_1608Metric
- D9: value LED -> D_Schottky; footprint LED_SMD:LED_0603_1608Metric -> Diode_SMD:D_SMA
- J1, J3, J7: footprint IoWLabsConnectors:Tb-2x1-5p-TH-V -> TerminalBlock_Phoenix:TerminalBlock_Phoenix_PT-1,5-2-3.5-H_1x02_P3.50mm_Horizontal
- J10: value HDR-2x1 -> HDR-4x1; footprint Connector_PinHeader_2.54mm:PinHeader_1x02_P2.54mm_Vertical -> TerminalBlock_Phoenix:TerminalBlock_Phoenix_PT-1,5-4-3.5-H_1x04_P3.50mm_Horizontal
- J14: value IN -> HDR-2x1; footprint IoWLabsConnectors:Tb-2x1-5p-TH-V -> TerminalBlock_Phoenix:TerminalBlock_Phoenix_PT-1,5-2-3.5-H_1x02_P3.50mm_Horizontal
- J15: value Conn_01x04 -> HDR-2x1; footprint Connector_JST:JST_XH_B4B-XH-AM_1x04_P2.50mm_Vertical -> TerminalBlock_Phoenix:TerminalBlock_Phoenix_PT-1,5-2-3.5-H_1x02_P3.50mm_Horizontal
- J16: value Conn_01x08 -> HDR-2x1; footprint Connector_JST:JST_XH_B8B-XH-AM_1x08_P2.50mm_Vertical -> TerminalBlock_Phoenix:TerminalBlock_Phoenix_PT-1,5-2-3.5-H_1x02_P3.50mm_Horizontal
- J17: value Micro_SD_Card -> HDR-2x1; footprint Connector_Card:microSD_HC_Wuerth_693072010801 -> TerminalBlock_Phoenix:TerminalBlock_Phoenix_PT-1,5-2-3.5-H_1x02_P3.50mm_Horizontal
- J18, J19: value HDR-3x1 -> HDR-2x1; footprint Jumper:SolderJumper-3_P1.3mm_Open_RoundedPad1.0x1.5mm_NumberLabels -> Connector_PinHeader_2.54mm:PinHeader_1x02_P2.54mm_Vertical
- J20: value HDR-4x1 -> IN; footprint IoWLabsConnectors:TB-4x1-5P-TH-V -> TerminalBlock_Phoenix:TerminalBlock_Phoenix_PT-1,5-2-3.5-H_1x02_P3.50mm_Horizontal
- J21: value HDR-4x1 -> Micro_SD_Card; footprint IoWLabsConnectors:TB-4x1-5P-TH-V -> Connector_Card:microSD_HC_Wuerth_693072010801
- J22: value HDR-4x1 -> Conn_01x08; footprint IoWLabsConnectors:TB-4x1-5P-TH-V -> Connector_JST:JST_XH_B8B-XH-AM_1x08_P2.50mm_Vertical
- J23: value HDR-4x1 -> Conn_01x08; footprint IoWLabsConnectors:TB-4x1-5P-TH-V -> Connector_JST:JST_XH_B6B-XH-AM_1x06_P2.50mm_Vertical
- J24, J25: value Conn_01x02 -> HDR-3x1; footprint Connector_JST:JST_XH_B2B-XH-AM_1x02_P2.50mm_Vertical -> Jumper:SolderJumper-3_P1.3mm_Open_RoundedPad1.0x1.5mm_NumberLabels
- J26: value Conn_01x02 -> HDR-4x1; footprint Connector_JST:JST_XH_B2B-XH-AM_1x02_P2.50mm_Vertical -> TerminalBlock_Phoenix:TerminalBlock_Phoenix_PT-1,5-4-3.5-H_1x04_P3.50mm_Horizontal
- J5: footprint IoWLabsConnectors:TB-4x1-5P-TH-V -> TerminalBlock_Phoenix:TerminalBlock_Phoenix_PT-1,5-4-3.5-H_1x04_P3.50mm_Horizontal
- J8: footprint IoWLabsConnectors:Tb-2x1-5p-TH-V -> Connector_JST:JST_XH_B2B-XH-A_1x02_P2.50mm_Vertical
- J9: footprint Connector_JST:JST_XH_B2B-XH-A_1x02_P2.50mm_Vertical -> Connector_PinHeader_2.54mm:PinHeader_1x02_P2.54mm_Vertical
- L2: value 33uH -> 4.7u; footprint Inductor_SMD:L_12x12mm_H8mm -> Inductor_SMD:L_Bourns_SRP7028A_7.3x6.6mm
- Q2: value Q_Dual_NPN_NPN_BRT_E1B1C2E2B2C1 -> Q_PMOS_GSD; footprint Package_TO_SOT_SMD:SOT-363_SC-70-6_Handsoldering -> Package_TO_SOT_SMD:SOT-23
- Q3: value Q_PMOS_GSD -> Q_Dual_NPN_NPN_BRT_E1B1C2E2B2C1; footprint Package_TO_SOT_SMD:SOT-23 -> Package_TO_SOT_SMD:SOT-363_SC-70-6_Handsoldering
- R24: value 10k -> 7k5
- R25, R37: value 10k -> 470
- R26: value 0 -> 10k
- R27: value 7k5 -> 10k
- R28: value 470 -> 0
- R36: value 10k -> 54.9k
- R38, R49, R50: value 1k -> 10k
- R40: value 3.3k -> 12k
- R41: value 12k -> 30k
- R42: value 30k -> 3.3k
- R44, R66, R68: value 3.3k -> 10k
- R46, R47, R48: value 10k -> 3.3k
- R51: value 1k -> 3.3k
- R52, R53, R54, R55: value 10k2 -> 10k
- R56, R57, R58, R59: value 3k3 -> 1k
- R63, R64: value 10k -> 1k
- R65, R70: value 3.3k -> 1k
- U10: value LM2596S-5 -> TPS562200; footprint Package_TO_SOT_SMD:TO-263-5_TabPin3 -> Package_TO_SOT_SMD:SOT-23-6
- U15: value MCP23017_SO -> PC817; footprint Package_SO:SOIC-28W_7.5x17.9mm_P1.27mm -> Package_DIP:DIP-4_W7.62mm
- moved JP9 204.5 mm to (77.5, 110.2), turned to 180 degrees
- moved C15 200.1 mm to (81.0, 48.8), turned to 90 degrees
- moved R38 197.4 mm to (87.5, 40.3), turned to 0 degrees
- moved R39 195.7 mm to (91.2, 48.4), turned to -90 degrees
- moved C14 189.9 mm to (83.0, 48.8), turned to 90 degrees
- moved D9 189.1 mm to (95.6, 46.5), turned to -90 degrees
- moved D10 187.4 mm to (117.5, 35.2), turned to 90 degrees
- moved L2 184.4 mm to (82.1, 38.2)
- moved D8 183.7 mm to (87.5, 37.1), turned to 0 degrees
- moved C13 175.4 mm to (81.0, 44.8)
- moved J11 168.3 mm to (111.2, 35.6), turned to 0 degrees
- moved U10 166.4 mm to (84.0, 45.0)
- moved C6 160.5 mm to (176.7, 51.3)
- moved R41 156.1 mm to (86.4, 49.0), turned to -90 degrees
- moved R40 152.6 mm to (84.9, 49.0), turned to -90 degrees
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Connections:
- C10 pad 1: RESET -> IO0
- C11 pad 1: Vbat_5V -> RESET
- C13 pad 1: VIN_12V -> Net-(U10-VBST)
- C13 pad 2: GND -> Net-(U10-SW)
- C14 pad 1: VIN_5V -> VIN_12V
- C15 pad 1: VIN_5V -> VIN_12V
- C24 pad 1: /VGPS_3V3 -> /VRFID_3V3
- C9 pad 1: IO0 -> Vbat_5V
- D10 pad 1: /Vpre_5V -> GND
- D10 pad 2: /V_USB -> Net-(D10-A)
- D8 pad 1: Net-(D8-K) -> GND
- D8 pad 2: GND -> Net-(D8-A)
- D9 pad 1: GND -> /Vpre_5V
- D9 pad 2: Net-(D9-A) -> /V_USB
- J10 pad 1: 12V_IN -> RS485_VDD_aux
- J10 pad 2: 420_VDD_ch2 -> RS485_VSS_aux
- J14 pad 1: VIN_12V -> 420_VDD_ch2
- J14 pad 2: GND -> 420_VSS_ch2
- J15 pad 1: GPA4 -> 420_sens_ch2+
- J15 pad 2: GPA5 -> 420_VSS_ch2
- J16 pad 1: GPB0 -> 420_VDD_ch1
- J16 pad 2: GPB1 -> 420_VSS_ch1
- J17 pad 1: unconnected-(J17-DAT2-Pad1) -> 420_sens_ch1+
- J17 pad 2: Net-(J17-DAT3/CD) -> 420_VSS_ch1
- J18 pad 1: +5V -> 12V_IN
- J18 pad 2: /EN_VS_S -> 420_VDD_ch2
- J19 pad 1: +5V -> 12V_IN
- J19 pad 2: /EN_VDL_S -> 420_VDD_ch1
- J21 pad 1: VIN_12V -> unconnected-(J21-DAT2-Pad1)
- J21 pad 2: GND -> Net-(J21-DAT3/CD)
- J21 pad 3: S2_IN -> Net-(J21-CMD)
- J21 pad 4: (no net) -> VDL_3V3
- J22 pad 1: VIN_12V -> +3V3
- J22 pad 2: GND -> Net-(J22-Pin_2)
- J22 pad 3: S3_IN -> GND
- J22 pad 4: (no net) -> IRQ
- J23 pad 1: VIN_12V -> +3V3
- J23 pad 3: S4_IN -> GPA4
- J23 pad 4: (no net) -> GPA5
- J24 pad 1: Net-(J24-Pin_1) -> +5V
- J24 pad 2: GND -> /EN_VS_S
- J25 pad 1: Net-(J25-Pin_1) -> +5V
- J25 pad 2: GND -> /EN_VDL_S
- J26 pad 1: Net-(J26-Pin_1) -> VIN_12V
- J7 pad 1: 420_sens_ch2_ -> RS485_VDD_aux
- J7 pad 2: 420_sens_ch2_+ -> RS485_VSS_aux
- J8 pad 1: 420_VDD_ch2 -> RESET
- J8 pad 2: 420_VSS_ch2 -> GND
- J9 pad 1: RESET -> 12V_IN
- J9 pad 2: GND -> RS485_VDD_aux
- JP6 pad 1: GND -> RS485_VSS_aux
- JP6 pad 2: 420_VSS_ch2 -> GND
- JP7 pad 1: +3V3 -> GND
- JP7 pad 2: A0 -> 420_VSS_ch2
- JP8 pad 1: +3V3 -> GND
- JP8 pad 2: A1 -> 420_VSS_ch1
- JP9 pad 2: A2 -> A0
- L2 pad 1: Net-(D8-K) -> Net-(U10-SW)
- Q2 pad 1: RST# -> /V_USB
- Q2 pad 2: Net-(Q2B-B1) -> /Vpre_5V
- Q2 pad 3: IO0 -> VIN_5V
- Q3 pad 1: /V_USB -> RST#
- Q3 pad 2: /Vpre_5V -> Net-(Q3B-B1)
- Q3 pad 3: VIN_5V -> IO0
- R18 pad 2: 420_VDD_ch2+ -> 420_sens_ch2+
- R19 pad 2: 420_VDD_ch1+ -> 420_sens_ch1+
- R24 pad 1: +3V3 -> Vbat_5V
- R24 pad 2: IO0 -> /FB_5V
- R25 pad 1: +3V3 -> Vbat_5V
- R25 pad 2: RESET -> Net-(D5-A)
- R26 pad 1: IO0 -> +3V3
- R26 pad 2: Net-(R26-Pad2) -> IO0
- R27 pad 1: Vbat_5V -> +3V3
- R27 pad 2: /FB_5V -> RESET
- R28 pad 1: Vbat_5V -> IO0
- R28 pad 2: Net-(D5-A) -> Net-(R28-Pad2)
- R36 pad 1: DTR# -> Net-(U10-VFB)
- R36 pad 2: Net-(Q2B-B1) -> VIN_5V
- R37 pad 1: Net-(Q2A-B1) -> VIN_5V
- R37 pad 2: RST# -> Net-(D8-A)
- R38 pad 1: Net-(D9-A) -> VIN_5V
- R38 pad 2: VIN_5V -> GND
- R40 pad 1: SPI1_MOSI -> V_AUTO_LVL
- R40 pad 2: Net-(J17-CMD) -> VIN_12V
- R41 pad 2: VIN_12V -> GND
- R42 pad 1: V_AUTO_LVL -> SPI1_MOSI
- R42 pad 2: GND -> Net-(J21-CMD)
- R43 pad 2: Net-(J17-CLK) -> Net-(J21-CLK)
- R44 pad 1: SD_CS -> Net-(J22-Pin_2)
- R44 pad 2: Net-(J17-DAT3/CD) -> SCL
- R45 pad 1: SPI1_MISO -> SD_CS
- R45 pad 2: Net-(J17-DAT0) -> Net-(J21-DAT3/CD)
- R46 pad 1: +3V3 -> Net-(J22-Pin_5)
- R46 pad 2: GPA0 -> SPI1_MISO
- R47 pad 1: +3V3 -> SPI1_MISO
- R47 pad 2: GPA1 -> Net-(J21-DAT0)
- R48 pad 1: +3V3 -> Net-(J22-Pin_6)
- R48 pad 2: GPA2 -> SPI1_MOSI
- R49 pad 1: Net-(J24-Pin_1) -> DTR#
- R49 pad 2: GPA0 -> Net-(Q3B-B1)
- R50 pad 1: Net-(J25-Pin_1) -> Net-(Q3A-B1)
- R50 pad 2: GPA1 -> RST#
- R51 pad 1: Net-(J26-Pin_1) -> Net-(J22-Pin_7)
- R51 pad 2: GPA2 -> SPI1_CLK
- R52 pad 1: S1_IN -> Net-(J22-Pin_8)
- R52 pad 2: SENSOR 1 -> SDA
- R53 pad 1: S2_IN -> +3V3
- R53 pad 2: SENSOR 2 -> GPA0
- R54 pad 1: S3_IN -> +3V3
- R54 pad 2: SENSOR 3 -> GPA1
- R55 pad 1: S4_IN -> +3V3
- R55 pad 2: SENSOR 4 -> GPA2
- R56 pad 1: GND -> +3V3
- R56 pad 2: SENSOR 1 -> Net-(D10-A)
- R57 pad 1: GND -> Net-(J30-Pin_1)
- R57 pad 2: SENSOR 2 -> GPA0
- R58 pad 1: GND -> Net-(J31-Pin_1)
- R58 pad 2: SENSOR 3 -> GPA1
- R59 pad 1: GND -> Net-(J32-Pin_1)
- R59 pad 2: SENSOR 4 -> GPA2
- R60 pad 2: Net-(D11-A) -> SENSOR 1
- R61 pad 1: VDL_3V3 -> +3V3
- R61 pad 2: Net-(D12-A) -> SENSOR 2
- R62 pad 1: /VGPS_3V3 -> +3V3
- R62 pad 2: Net-(D13-A) -> SENSOR 3
- R63 pad 1: SDA -> +3V3
- R63 pad 2: Net-(U15-SDA) -> SENSOR 4
- R64 pad 1: SCL -> VDL_3V3
- R64 pad 2: Net-(U15-SCK) -> Net-(D11-A)
- R65 pad 1: MCP_RESET -> /VRFID_3V3
- R65 pad 2: +3V3 -> Net-(D12-A)
- R66 pad 1: INTA -> SCL
- R66 pad 2: +3V3 -> Net-(U19-SCL)
- R67 pad 1: INTB -> MCP_RESET
- R68 pad 1: GND -> SDA
- R68 pad 2: A0 -> Net-(U19-SDA)
- R69 pad 1: GND -> INTA
- R69 pad 2: A1 -> +3V3
- R70 pad 1: GND -> S1_IN
- R70 pad 2: A2 -> Net-(R70-Pad2)
- R9 pad 1: /Data_B -> RS485_B_ch2
- R9 pad 2: /Data_A -> RS485_A_ch2
- SW3 pad 3: Net-(R26-Pad2) -> Net-(R28-Pad2)
- SW3 pad 4: Net-(R26-Pad2) -> Net-(R28-Pad2)
- U10 pad 1: VIN_12V -> GND
- U10 pad 2: Net-(D8-K) -> Net-(U10-SW)
- U10 pad 3: GND -> VIN_12V
- U10 pad 4: VIN_5V -> Net-(U10-VFB)
- U10 pad 5: GND -> VIN_12V
- U14 pad 5: /VGPS_3V3 -> /VRFID_3V3
- U15 pad 1: GPB0 -> Net-(R70-Pad2)
- U15 pad 2: GPB1 -> GND
- U15 pad 3: GPB2 -> GND
- U15 pad 4: GPB3 -> SENSOR 1
- U2 pad 6: /Data_A -> RS485_A_ch2
- U2 pad 7: /Data_B -> RS485_B_ch2
- U6 pad 7: 420_VDD_ch2+ -> 420_sens_ch2+
- U7 pad 7: 420_VDD_ch1+ -> 420_sens_ch1+
Other:
- board outline added: 130 x 100 mm
- board text added: "12+"
- board text added: "12-"
- board text added: "12V"
- board text added: "3V3"
- board text added: "B+"
- board text added: "B-"
- board text added: "B1"
- board text added: "B2"
- board text added: "B3"
- board text added: "GND"
- board text added: "IRQ"
- board text added: "MI"
- board text added: "MO"
- board text added: "S1"
- board text added: "S2"
- board text added: "S3"
- board text added: "S4"
- board text added: "SCK"
- board text added: "SCL"
- board text added: "SDA"
